Commit message: File system update:

File: models/virat/virat_model.xacro (robot description, xacro)
@@ -1,19 +1,13 @@
-<?xml version="1.0" ?>
-<<<<<<< HEAD
-<robot name="virat">
-    <link name="base_link">
-        <inertial>
-            <origin xyz="0 0 0" rpy="0 0 0"/>
-            <mass value="5"/>
-            <inertia ixx="0.005" ixy="0.005" ixz="0.005" iyy="0.005" iyz="0.005" izz="0.005"/>
-=======
-<robot name="clueless_virat">
+<?xml version='1.0'?>
+<robot name="clueless_virat" xmlns:xacro="http://www.ros.org/wiki/xacro">
+  <xacro:property name="cameraSize" value="0.05"/>
+  <xacro:property name="cameraMass" value="0.1"/>
+  <xacro:include filename="$(find virat_gazebo)/models/virat/virat.gazebo" />
     <static>false</static>
     <link name="base_link">
         <inertial>
             <origin xyz="0 0 0" rpy="0 0 0"/>
-            <mass value="0.5"/>
-            <inertia ixx="0.05" ixy="0.05" ixz="0.05" iyy="0.05" iyz="0.05" izz="0.05"/>
->>>>>>> 3f20f738ae0f54869a4eaa44299b4808d3346e59
+            <mass value="2"/>
+            <inertia ixx="0.001" ixy="0" ixz="0" iyy="0.001" iyz="0" izz="0.001"/>
         </inertial>
         <visual>
@@ -30,6 +24,7 @@
         </collision>
     </link>
-    <!-- =====================Left Wheel======================-->
-    <link name="left_wheel">
+    <!-- =====================Wheels======================-->
+    <xacro:macro name="wheel" params="prefix reflect">
+    <link name="${prefix}_wheel">
         <visual>
             <origin xyz="0 0 0" rpy="0 0 0"/>
@@ -40,10 +35,6 @@
         <inertial>
             <origin xyz="0 0 0" rpy="0 0 0"/>
-<<<<<<< HEAD
-            <mass value="0.5"/>
-=======
             <mass value="0.05"/>
->>>>>>> 3f20f738ae0f54869a4eaa44299b4808d3346e59
-            <inertia ixx="0.005" ixy="0.005" ixz="0.005" iyy="0.005" iyz="0.005" izz="0.005"/>
+            <inertia ixx="0.001" ixy="0" ixz="0" iyy="0.001" iyz="0" izz="0.001"/>
         </inertial>
         <collision>
@@ -54,36 +45,13 @@
         </collision>
     </link>
-    <joint name="left_wheel_joint" type="continuous">
+    <joint name="${prefix}_wheel_joint" type="continuous">
         <parent link="base_link"/>
-        <child link="left_wheel"/>
-        <origin xyz="0 0.323 0" rpy="0 0 0"/>
+        <child link="${prefix}_wheel"/>
+        <origin xyz="0 ${reflect*0.323} 0" rpy="0 0 0"/>
         <axis xyz="0 1 0"/>
     </joint>
-    <!-- =====================Right Wheel======================-->
-    <link name="right_wheel">
-        <visual>
-            <origin xyz="0 0 0" rpy="0 0 0"/>
-                <geometry>
-                    <mesh filename="package://virat_gazebo/models/virat/meshes/tyre1.dae"/>
-                </geometry>
-        </visual>
-        <inertial>
-            <origin xyz="0 0 0" rpy="0 0 0"/>
-            <mass value="0.5"/>
-            <inertia ixx="0.05" ixy="0.05" ixz="0.05" iyy="0.05" iyz="0.05" izz="0.05"/>
-        </inertial>
-        <collision>
-            <origin xyz="0 0 0" rpy="0 0 0"/>
-                <geometry>
-                    <mesh filename="package://virat_gazebo/models/virat/meshes/tyre1.dae"/>
-                </geometry>
-        </collision>
-    </link>
-    <joint name="right_wheel_joint" type="continuous">
-        <parent link="base_link"/>
-        <child link="right_wheel"/>
-        <origin xyz="0 -0.323 0" rpy="0 0 0"/>
-        <axis xyz="0 1 0"/>
-    </joint>
+    </xacro:macro>
+    <xacro:wheel prefix="right" reflect="1" />
+    <xacro:wheel prefix="left" reflect="-1" />
     <!-- =====================Castor Wheel======================-->
     <link name="connect_castor_link">
@@ -97,5 +65,5 @@
             <origin xyz="0 0 0" rpy="0 0 0"/>
             <mass value="0.5"/>
-            <inertia ixx="0.05" ixy="0.05" ixz="0.05" iyy="0.05" iyz="0.05" izz="0.05"/>
+            <inertia ixx="0.001" ixy="0" ixz="0" iyy="0.001" iyz="0" izz="0.001"/>
         </inertial>
         <collision>
@@ -116,24 +84,16 @@
             <origin xyz="0 0 0 " rpy="0 0 0"/>
                 <geometry>
-<<<<<<< HEAD
-                    <mesh filename="package://virat_gazebo/models/virat/meshes/castors1.dae"/>
-=======
                     <mesh filename="package://virat_gazebo/models/virat/meshes/castors1.dae" scale="1.45 1.45 1.45"/>
->>>>>>> 3f20f738ae0f54869a4eaa44299b4808d3346e59
                 </geometry>
         </visual>
         <inertial>
             <origin xyz="0 0 0" rpy="0 0 0"/>
-            <mass value="0.5"/>
-            <inertia ixx="0.05" ixy="0.05" ixz="0.05" iyy="0.05" iyz="0.05" izz="0.05"/>
+            <mass value="2"/>
+            <inertia ixx="0.001" ixy="0" ixz="0" iyy="0.001" iyz="0" izz="0.001"/>
         </inertial>
         <collision>
             <origin xyz="0 0 0 " rpy="0 0 0"/>
                 <geometry>
-<<<<<<< HEAD
-                    <mesh filename="package://virat_gazebo/models/virat/meshes/castors1.dae"/>
-=======
                     <mesh filename="package://virat_gazebo/models/virat/meshes/castors1.dae" scale="1.45 1.45 1.45"/>
->>>>>>> 3f20f738ae0f54869a4eaa44299b4808d3346e59
                 </geometry>
         </collision>
@@ -145,3 +105,35 @@
         <axis xyz="0 0 0"/>
     </joint>
+ <!-- =========================Cameras======================================= -->
+ <xacro:macro name="camera" params="prefix reflect">
+ <link name="${prefix}_camera">
+    <collision>
+      <origin xyz="0 0 0" rpy="0 0 0"/>
+      <geometry>
+        <box size="${cameraSize} ${cameraSize} ${cameraSize}"/>
+      </geometry>
+    </collision>
+    <visual>
+      <origin xyz="0 0 0" rpy="0 0 0"/>
+      <geometry>
+        <box size="${cameraSize} ${cameraSize} ${cameraSize}"/>
+      </geometry>
+      <material name="green"/>
+    </visual>
+    <inertial>
+      <mass value="${cameraMass}" />
+      <origin xyz="0 0 0" rpy="0 0 0"/>
+      <box_inertia m="${cameraMass}" x="${cameraSize}" y="${cameraSize}" z="${cameraSize}" />
+      <inertia ixx="1e-6" ixy="0" ixz="0" iyy="1e-6" iyz="0" izz="1e-6" />
+    </inertial>
+  </link>
+  <joint name="${prefix}_camera_joint" type="fixed">
+    <axis xyz="0 1 0" />
+    <origin xyz="0.72 ${reflect*0.05} 1.175" rpy="0 0 0"/>
+    <parent link="base_link"/>
+    <child link="${prefix}_camera"/>
+  </joint>
+</xacro:macro>
+<xacro:camera prefix="right" reflect="1"/>
+<xacro:camera prefix="left" reflect="-1"/>
 </robot>

Commit message: tuned masses and diff drive properties due to excessive tyre slipping

File: models/virat/virat_model.xacro (robot description, xacro)
@@ -2,5 +2,5 @@
 <robot name="clueless_virat" xmlns:xacro="http://www.ros.org/wiki/xacro">
   <xacro:property name="cameraSize" value="0.05"/>
-  <xacro:property name="cameraMass" value="0.1"/>
+  <xacro:property name="cameraMass" value="0.01"/>
   <xacro:include filename="$(find virat_gazebo)/models/virat/virat.gazebo" />
     <static>false</static>
@@ -8,5 +8,5 @@
         <inertial>
             <origin xyz="0 0 0" rpy="0 0 0"/>
-            <mass value="2"/>
+            <mass value="1.5"/>
             <inertia ixx="0.001" ixy="0" ixz="0" iyy="0.001" iyz="0" izz="0.001"/>
         </inertial>
@@ -35,5 +35,5 @@
         <inertial>
             <origin xyz="0 0 0" rpy="0 0 0"/>
-            <mass value="0.05"/>
+            <mass value="0.4"/>
             <inertia ixx="0.001" ixy="0" ixz="0" iyy="0.001" iyz="0" izz="0.001"/>
         </inertial>
@@ -51,36 +51,7 @@
         <axis xyz="0 1 0"/>
     </joint>
-<<<<<<< HEAD:models/virat/virat_model.urdf
-    <!-- =====================Right Wheel======================-->
-    <link name="right_wheel">
-        <visual>
-            <origin xyz="0 0 0" rpy="0 0 0"/>
-                <geometry>
-                    <mesh filename="package://virat_gazebo/models/virat/meshes/tyre1.dae"/>
-                </geometry>
-        </visual>
-        <inertial>
-            <origin xyz="0 0 0" rpy="0 0 0"/>
-            <mass value="0.5"/>
-            <inertia ixx="0.001" ixy="0" ixz="0" iyy="0.001" iyz="0" izz="0.001"/>
-        </inertial>
-        <collision>
-            <origin xyz="0 0 0" rpy="0 0 0"/>
-                <geometry>
-                    <mesh filename="package://virat_gazebo/models/virat/meshes/tyre1.dae"/>
-                </geometry>
-        </collision>
-    </link>
-    <joint name="right_wheel_joint" type="continuous">
-        <parent link="base_link"/>
-        <child link="right_wheel"/>
-        <origin xyz="0 -0.323 0" rpy="0 0 0"/>
-        <axis xyz="0 1 0"/>
-    </joint>
-=======
     </xacro:macro>
     <xacro:wheel prefix="right" reflect="1" />
     <xacro:wheel prefix="left" reflect="-1" />
->>>>>>> 92df7c5a3a0190f917eccf8c6d7cae76888ac12d:models/virat/virat_model.xacro
     <!-- =====================Castor Wheel======================-->
     <link name="connect_castor_link">
@@ -118,11 +89,6 @@
         <inertial>
             <origin xyz="0 0 0" rpy="0 0 0"/>
-<<<<<<< HEAD:models/virat/virat_model.urdf
-            <mass value="0.5"/>
-            <inertia ixx="0.001" ixy=".05" ixz="0" iyy="0.001" iyz="0" izz="0.001"/>
-=======
-            <mass value="2"/>
+            <mass value="1"/>
             <inertia ixx="0.001" ixy="0" ixz="0" iyy="0.001" iyz="0" izz="0.001"/>
->>>>>>> 92df7c5a3a0190f917eccf8c6d7cae76888ac12d:models/virat/virat_model.xacro
         </inertial>
         <collision>
@@ -139,29 +105,4 @@
         <axis xyz="0 0 0"/>
     </joint>
-<<<<<<< HEAD:models/virat/virat_model.urdf
-    <gazebo>
-        <plugin name="differential_drive_controller" filename="libgazebo_ros_diff_drive.so">
-            <commandTopic>/cmd_vel</commandTopic>
-            <odometryTopic>/odom</odometryTopic>
-            <odometryFrame>odom</odometryFrame>
-            <odometrySource>world</odometrySource>
-            <publishOdomTF>true</publishOdomTF>
-            <robotBaseFrame>base_link</robotBaseFrame>
-            <publishWheelTF>false</publishWheelTF>
-            <publishTf>true</publishTf>
-            <publishWheelJointState>true</publishWheelJointState>
-            <legacyMode>false</legacyMode>
-            <updateRate>30</updateRate>
-            <leftJoint>left_wheel_joint</leftJoint>
-            <rightJoint>right_wheel_joint</rightJoint>
-            <wheelSeparation>0.65</wheelSeparation>
-            <wheelDiameter>0.4</wheelDiameter>
-            <wheelAcceleration>1</wheelAcceleration>
-            <wheelTorque>10</wheelTorque>
-            <rosDebugLevel>na</rosDebugLevel>
-        </plugin>
-    </gazebo>
-</robot>
-=======
  <!-- =========================Cameras======================================= -->
  <xacro:macro name="camera" params="prefix reflect">
@@ -197,3 +138,2 @@
 <xacro:camera prefix="left" reflect="-1"/>
 </robot>
->>>>>>> 92df7c5a3a0190f917eccf8c6d7cae76888ac12d:models/virat/virat_model.xacro

Commit message: added lidar

File: models/virat/virat_model.xacro (robot description, xacro)
@@ -137,3 +137,29 @@
 <xacro:camera prefix="right" reflect="1"/>
 <xacro:camera prefix="left" reflect="-1"/>
+<!-- =========================Laser======================================= -->
+<link name="hokuyo">
+    <collision>
+      <origin xyz="0 0 0" rpy="0 0 0"/>
+      <geometry>
+    <box size="0.1 0.1 0.1"/>
+      </geometry>
+    </collision>
+    <visual>
+      <origin xyz="0 0 0" rpy="0 0 0"/>
+      <geometry>
+        <mesh filename="package://virat_gazebo/models/virat/meshes/sick-lms1xx.dae"/>
+      </geometry>
+    </visual>
+    <inertial>
+      <mass value="1e-5" />
+      <origin xyz="0 0 0" rpy="0 0 0"/>
+      <inertia ixx="1e-6" ixy="0" ixz="0" iyy="1e-6" iyz="0" izz="1e-6" />
+    </inertial>
+</link>
+  <joint name="hokuyo_joint" type="fixed">
+    <axis xyz="0 1 0" />
+    <origin xyz="0.76 0 0.39" rpy="0 0 0"/>
+    <parent link="base_link"/>
+    <child link="hokuyo"/>
+  </joint>
 </robot>

Commit message: tweaked lidar params for gmapping

File: models/virat/virat_model.xacro (robot description, xacro)
@@ -156,5 +156,5 @@
       <inertia ixx="1e-6" ixy="0" ixz="0" iyy="1e-6" iyz="0" izz="1e-6" />
     </inertial>
-</link>
+  </link>
   <joint name="hokuyo_joint" type="fixed">
     <axis xyz="0 1 0" />

Commit message: Updated inertial values

File: models/virat/virat_model.xacro (robot description, xacro)
@@ -9,5 +9,5 @@
             <origin xyz="0 0 0" rpy="0 0 0"/>
             <mass value="1.5"/>
-            <inertia ixx="0.001" ixy="0" ixz="0" iyy="0.001" iyz="0" izz="0.001"/>
+            <inertia ixx="0.001459" ixy="0.004549" ixz="0.002897" iyy="0.012432" iyz="-0.000924" izz="0.012627"/>
         </inertial>
         <visual>

Commit message: added dummy link: fix melodic issue

File: models/virat/virat_model.xacro (robot description, xacro)
@@ -5,4 +5,5 @@
   <xacro:include filename="$(find virat_gazebo)/models/virat/virat.gazebo" />
     <static>false</static>
+    <link name="dummy"> </link>
     <link name="base_link">
         <inertial>
@@ -24,4 +25,8 @@
         </collision>
     </link>
+      <joint name="dummy_joint" type="fixed">
+      <parent link="dummy" />
+      <child link="base_link" />
+    </joint>
     <!-- =====================Wheels======================-->
     <xacro:macro name="wheel" params="prefix reflect">

Commit message: fixed tf issue of base footprint

File: models/virat/virat_model.xacro (robot description, xacro)
@@ -5,5 +5,10 @@
   <xacro:include filename="$(find virat_gazebo)/models/virat/virat.gazebo" />
     <static>false</static>
-    <link name="dummy"> </link>
+  <link name="base_footprint"/>
+  <joint name="base_joint" type="fixed">
+    <parent link="base_footprint"/>
+    <child link="base_link"/>
+    <origin xyz="0.0 0.0 0.010" rpy="0 0 0"/>
+  </joint>
     <link name="base_link">
         <inertial>
@@ -25,8 +30,4 @@
         </collision>
     </link>
-      <joint name="dummy_joint" type="fixed">
-      <parent link="dummy" />
-      <child link="base_link" />
-    </joint>
     <!-- =====================Wheels======================-->
     <xacro:macro name="wheel" params="prefix reflect">
